File: Arduinio Clone.kicad_sch (KiCad schematic)
At the start: 13 parts, among them U1 DS1337_GM, U2 24LC1025, U3 ATmega328P-A, U4 24LC1025, Y1 Crystal 32MHz, Y2 Crystal 16MHz

Commit message: ERC run
Connections:
- no-connect marks 9 -> 8
Other:
- moved on the sheet: BT1, C1, C2, C3, D1, R1, R2, U3, Y2

Commit message: Started working on PCB new
Changed lines of the file:
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@@
+    (stroke (width 0) (type default) (color 0 0 0 0))
+  )
+  (polyline (pts (xy 123.19 125.73) (xy 279.4 125.73))
+    (stroke (width 0) (type default) (color 0 0 0 0))
+  )
+  (polyline (pts (xy 82.55 81.28) (xy 82.55 34.29))
     (stroke (width 0) (type default) (color 0 0 0 0))
   )
@@
     (stroke (width 0) (type default) (color 0 0 0 0))
   )
+  (polyline (pts (xy 123.19 22.86) (xy 123.19 33.02))
+    (stroke (width 0) (type default) (color 0 0 0 0))
+  )
   (wire (pts (xy 158.75 162.56) (xy 161.29 162.56))
     (stroke (width 0) (type default) (color 0 0 0 0))
@@
     (stroke (width 0) (type default) (color 0 0 0 0))
   )
+  (polyline (pts (xy 13.97 81.28) (xy 13.97 34.29))
+    (stroke (width 0) (type default) (color 0 0 0 0))
+  )
   (wire (pts (xy 31.75 46.99) (xy 40.64 46.99))
     (stroke (width 0) (type default) (color 0 0 0 0))
@@
     (stroke (width 0) (type default) (color 0 0 0 0))
   )
+  (polyline (pts (xy 279.4 22.86) (xy 123.19 22.86))
+    (stroke (width 0) (type default) (color 0 0 0 0))
+  )
   (wire (pts (xy 31.75 57.15) (xy 31.75 59.69))
     (stroke (width 0) (type default) (color 0 0 0 0))
@@
     (stroke (width 0) (type default) (color 0 0 0 0))
   )
+  (polyline (pts (xy 279.4 125.73) (xy 279.4 22.86))
+    (stroke (width 0) (type default) (color 0 0 0 0))
+  )
+  (polyline (pts (xy 123.19 27.94) (xy 123.19 125.73))
+    (stroke (width 0) (type default) (color 0 0 0 0))
+  )
   (wire (pts (xy 158.75 149.86) (xy 161.29 149.86))
     (stroke (width 0) (type default) (color 0 0 0 0))
@@
     (stroke (width 0) (type default) (color 0 0 0 0))
   )
+  (polyline (pts (xy 13.97 34.29) (xy 82.55 34.29))
+    (stroke (width 0) (type default) (color 0 0 0 0))
+  )
   (wire (pts (xy 40.64 57.15) (xy 40.64 59.69))
     (stroke (width 0) (type default) (color 0 0 0 0))
@@
     (stroke (width 0) (type default) (color 0 0 0 0))
   )
+  (polyline (pts (xy 82.55 34.29) (xy 80.01 34.29))
+    (stroke (width 0) (type default) (color 0 0 0 0))
+  )
   (wire (pts (xy 176.53 59.69) (xy 193.04 59.69))
     (stroke (width 0) (type default) (color 0 0 0 0))
@@
   )
   (wire (pts (xy 76.2 97.79) (xy 76.2 91.44))
+    (stroke (width 0) (type default) (color 0 0 0 0))
+  )
+  (polyline (pts (xy 82.55 81.28) (xy 13.97 81.28))
     (stroke (width 0) (type default) (color 0 0 0 0))
   )
@@
   (symbol (lib_id "power:PWR_FLAG") (at 39.37 128.27 270) (unit 1)
     (in_bom yes) (on_board yes) (fields_autoplaced)
-    (property "Reference" "#FLG?" (id 0) (at 41.275 128.27 0)
+    (property "Reference" "#FLG02" (id 0) (at 41.275 128.27 0)
       (effects (font (size 1.27 1.27)) hide)
     )
@@
     )
     (path "/0cb03926-b122-4cdb-83ee-3a07cc2bdb27"
-      (reference "#FLG?") (unit 1) (value "PWR_FLAG") (footprint "")
+      (reference "#FLG02") (unit 1) (value "PWR_FLAG") (footprint "")
     )
     (path "/0c152b16-db1d-4916-8114-a71f273967e1"
