File: Arduinio Clone_4_layer.kicad_pcb (KiCad board)
At the start: 4 copper layers, 50.8 x 25.4 mm, 17 parts, among them J1 Serial, J2 Digital Pins, J3 ICSP, J4 I2C, U1 DS1337_GM, U2 24LC1025, U3 ATmega328P-A, U4 24LC1025, Y1 Crystal 32MHz, Y2 Crystal 16MHz

Commit message: Saved fully routed 4 layer board
Routing:
- net /VCC: track 0.00 -> 139.7 mm
- net GNDPWR: track 0.00 -> 128.8 mm, vias 0 -> 1
- net /SCK: track 0.00 -> 84.5 mm, vias 0 -> 1
- net /SDA: track 0.00 -> 46.3 mm, vias 0 -> 2
- net /MISO: track 0.00 -> 43.2 mm
- net /RESET: track 0.00 -> 33.5 mm
- net /D2: track 0.00 -> 27.4 mm
- net /MOSI: track 0.00 -> 27.1 mm, vias 0 -> 1
- net /ADDR2: track 0.00 -> 21.1 mm
- net /D3: track 0.00 -> 13.4 mm, vias 0 -> 1
- net /D4: track 0.00 -> 12.8 mm, vias 0 -> 1
- net /RX: track 0.00 -> 12.6 mm, vias 0 -> 1
- net Net-(C1-Pad2): track 0.00 -> 11.9 mm
- net /ADDR1: track 0.00 -> 10.9 mm
- net Net-(U1-Pad1): track 0.00 -> 10.0 mm
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