File: Arduinio Clone_2_layer.kicad_pcb (KiCad board)
At the start: 2 copper layers, 50.8 x 25.4 mm, 17 parts, among them J1 Serial, J2 Digital Pins, J3 ICSP, J4 I2C, U1 DS1337_GM, U2 24LC1025, U3 ATmega328P-A, U4 24LC1025, Y1 Crystal 32MHz, Y2 Crystal 16MHz

Commit message: Added Back silkscreen text
Other:
- board text added: "Designed by Giddie"
Changed lines of the file:
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@@
   (layers
     (0 "F.Cu" signal)
-    (31 "B.Cu" signal)
+    (31 "B.Cu" power)
     (32 "B.Adhes" user "B.Adhesive")
     (33 "F.Adhes" user "F.Adhesive")
@@
   (gr_circle (center 142.24 81.28) (end 142.24 82.55) (layer "Edge.Cuts") (width 0.1) (fill none))
   (gr_arc (start 144.780001 101.600001) (mid 144.036052 103.396052) (end 142.240001 104.140001) (layer "Edge.Cuts") (width 0.1))
+  (gr_text "Designed by Giddie\n" (at 124.46 92.71) (layer "B.SilkS")
+    (effects (font (size 1 1) (thickness 0.15)) (justify mirror))
+  )
   (segment (start 134.4508 89.535) (end 134.93 89.535) (width 0.3) (layer "F.Cu") (net 1))
   (segment (start 132.6503 100.3997) (end 135.26 97.79) (width 0.3) (layer "F.Cu") (net 1))
